File: KiCAD/8Bit_EuroRack.kicad_pcb (KiCad board)
At the start: 2 copper layers, 25.2 x 128.5 mm, 32 parts, among them J4 Con_3-5V, J6 Sync_Jumper, SW2 SW_Push, SW3 SW_Push, SW4 SW_Push, U1 ATTINY85-20SU

Commit message: adding screenshots
Parts:
- added REF**: PJ301M-12, 8Bit_Eurorack:PJ301M-12, F.Cu at (51.8, 83.0)
Changed lines of the file:
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@@
     (tracks 264)
     (zones 0)
-    (modules 32)
+    (modules 33)
     (nets 19)
   )
@@
     (uvia_drill 0.1)
   )
+  (module 8Bit_Eurorack:PJ301M-12 (layer F.Cu)
+    (at 51.82 82.96)
+    (fp_text reference REF** (at 4.064 5.588) (layer F.SilkS)
+      (effects (font (size 1 1) (thickness 0.15)))
+    )
+    (fp_text value PJ301M-12 (at 0 -7.112) (layer F.Fab)
+      (effects (font (size 1 1) (thickness 0.15)))
+    )
+    (fp_line (start -4.5 -6.2) (end 4.5 -6.2) (layer F.SilkS) (width 0.15))
+    (fp_line (start -4.5 4.7) (end 4.5 4.7) (layer F.SilkS) (width 0.15))
+    (fp_line (start -4.5 -6.2) (end -4.5 4.7) (layer F.SilkS) (width 0.15))
+    (fp_line (start 4.5 -6.2) (end 4.5 4.7) (layer F.SilkS) (width 0.15))
+    (fp_circle (center 0 0) (end 1.8 0) (layer F.SilkS) (width 0.15))
+    (fp_line (start 0 -1.8) (end 0 1.8) (layer F.SilkS) (width 0.15))
+    (fp_line (start -1.8 0) (end 1.8 0) (layer F.SilkS) (width 0.15))
+    (pad 3 thru_hole circle (at 0 -4.92) (size 1.8 1.8) (drill 1.6) (layers *.Cu *.Mask F.SilkS))
+    (pad 1 thru_hole circle (at 0 6.48) (size 1.8 1.8) (drill 1.6) (layers *.Cu *.Mask F.SilkS))
+    (pad 2 thru_hole circle (at 0 3.38) (size 1.8 1.8) (drill 1.6) (layers *.Cu *.Mask F.SilkS))
+    (model :stahllabs:PJ301M-12.step
+      (at (xyz 0 0 0))
+      (scale (xyz 1 1 1))
+      (rotate (xyz 0 0 0))
+    )
+  )
   (module 8Bit_Eurorack:SW_SPST_FSMSM (layer F.Cu)
     (at 78.97 95.65 180)
@@
       (rotate (xyz 0 0 0))
     )
+    (model /usr/share/kicad/modules/packages3d/Resistor_SMD.3dshapes/R_1206_3216Metric.step
+      (at (xyz 0 0 0))
+      (scale (xyz 1 1 1))
+      (rotate (xyz 0 0 0))
+    )
   )
   (module 8Bitmixtape_reworked:R_1206_HandSoldering (layer B.Cu)
@@
       (at (xyz 0 0 0))
       (scale (xyz 1 1 1))
+      (rotate (xyz 0 0 0))
+    )
+    (model /usr/share/kicad/modules/packages3d/Package_DIP.3dshapes/DIP-8_W7.62mm.step
+      (at (xyz 0 0 0))
+      (scale (xyz 1 1 1))

Commit message: adding photos
Parts:
- removed REF**: PJ301M-12, 8Bit_Eurorack:PJ301M-12
